File: hw/pcb/rgb-lamp/rgb-lamp.kicad_pcb (KiCad board)
At the start: 2 copper layers, 64.3 x 65 mm, 15 parts, among them J1 Conn_01x04_Socket, J2 Conn_01x02_Socket, Q1 NMOS, Q2 NMOS, Q3 NMOS, U1 Pico

Commit message: Add more docs
Parts:
- added J3: Rotary_Encoder_Connector, Connector_JST:JST_XH_B4B-XH-A_1x04_P2.50mm_Vertical, F.Cu at (80.1, 93.3)
- added R4: 10k, Resistor_THT:R_Axial_DIN0207_L6.3mm_D2.5mm_P10.16mm_Horizontal, F.Cu at (43.3, 51.2)
- added R5: 10k, Resistor_THT:R_Axial_DIN0207_L6.3mm_D2.5mm_P10.16mm_Horizontal, F.Cu at (51.7, 55.5)
- added R6: 10k, Resistor_THT:R_Axial_DIN0207_L6.3mm_D2.5mm_P10.16mm_Horizontal, F.Cu at (58.3, 72.2)
- J1: value Conn_01x04_Socket -> RGB_Strip_Connector
- R1, R2, R3: value 100 -> 220
- moved Q3 14.7 mm to (57.0, 67.2), turned to 0 degrees
- moved R2 13.6 mm to (49.9, 41.5)
- moved Q2 10.7 mm to (50.4, 50.5), turned to 0 degrees
- moved R1 10.6 mm to (50.4, 36.4)
- moved J1 10.0 mm to (46.9, 73.9), turned to -90 degrees
- moved R3 9.23 mm to (58.5, 58.8), turned to 90 degrees
- moved U1 9.06 mm to (75.8, 60.6)
- moved Q1 2.19 mm to (41.8, 45.7), turned to 0 degrees
Connections:
- U1 pad 17: unconnected-(U1-GPIO13-Pad17)_1 -> Net-(J3-DT)
- U1 pad 19: unconnected-(U1-GPIO14-Pad19)_1 -> Net-(J3-CLK)
- U1 pad 20: unconnected-(U1-GPIO15-Pad20) -> Net-(J3-Switch)
Routing:
- net Net-(J3-DT): track 0.00 -> 31.3 mm
- net Net-(J3-CLK): track 0.00 -> 28.5 mm
- net Net-(J3-Switch): track 0.00 -> 12.8 mm
- net Net-(Q1-G): track 8.37 -> 17.9 mm
- net Net-(Q2-G): track 8.62 -> 14.7 mm
- net Net-(J1-B): track 12.9 -> 18.4 mm
- net Net-(J1-R): track 39.2 -> 33.9 mm
- net Net-(Q3-G): track 9.25 -> 13.6 mm
- net +5V: track 27.9 -> 30.7 mm
- net Net-(U1-GPIO2): track 13.1 -> 10.3 mm
- net Net-(U1-GPIO1): track 10.0 -> 7.91 mm
- net Net-(U1-GPIO0): track 7.58 -> 6.35 mm
- net Net-(J1-G): track 30.4 -> 31.1 mm
