File: hw/pcb/rgb-lamp/rgb-lamp.kicad_sch (KiCad schematic)
At the start: 11 parts, among them J1 Conn_01x04_Socket, J2 Conn_01x02_Socket, Q1 NMOS, Q2 NMOS, Q3 NMOS, U1 Pico

Commit message: Add more docs
Parts:
- added J3: Rotary_Encoder_Connector, Connector_JST:JST_XH_B4B-XH-A_1x04_P2.50mm_Vertical, symbol Connector:Conn_01x04_Pin
- added R4, R5, R6: 10k, Resistor_THT:R_Axial_DIN0207_L6.3mm_D2.5mm_P10.16mm_Horizontal, symbol Device:R
- J1: value Conn_01x04_Socket -> RGB_Strip_Connector
- R1, R2, R3: value 100 -> 220
Connections:
- net GND: now also J3.4 (GND), R4.2, R5.2, R6.2
- net at Q3.2 (G), R3.1: now also R6.1
- net at Q2.2 (G), R2.1: now also R5.1
- net at U1.17 (GPIO13): now also J3.1 (DT)
- net at U1.19 (GPIO14): now also J3.2 (CLK)
- net at U1.20 (GPIO15): now also J3.3 (Switch)
- net at Q1.2 (G), R1.1: now also R4.1
- no-connect marks 38 -> 35
